Commit message: Some fixes

File: m2wr_description/urdf/gazebo_control.xacro (robot description, xacro)
@@ -8,14 +8,12 @@
                 <wheel_separation>0.35</wheel_separation>
                 <wheel_diameter>0.1</wheel_diameter>
-            <!-- Connector inf -->
-                <element2_link_joint>element2_link_joint</element2_link_joint>
             <!-- limits -->
                 <max_wheel_torque>200</max_wheel_torque>
                 <max_acceleration>10.0</max_acceleration>
             <!-- Output -->
+                <odometry_topic>odom</odometry_topic>
                 <odometry_frame>odom</odometry_frame>
                 <robot_base_frame>base_footprint</robot_base_frame>
-                <robot_base_frame_2>base_link_2</robot_base_frame_2>
-                <publish_rate>50</publish_rate>
+                <update_rate>50</update_rate>
                 <publish_odom>true</publish_odom>
                 <publish_odom_tf>true</publish_odom_tf>

File: m2wr_description/urdf/lidar.xacro (robot description, xacro)
@@ -4,5 +4,5 @@
         <parent link="chassis"/>
         <child link="laser_frame"/>
-        <origin xyz="0.122 0 0.212" rpy="0 0 0"/>
+        <origin xyz="0.25 0 0.212" rpy="0 0 0"/>
     </joint>
     <link name="laser_frame">

File: spherorobot_cpp/urdf/spherorobot_v5_1.urdf (robot description, URDF)
Before this commit: robot spherorobot_v5_1, 3 links, 2 joints
Links:
- link base_link: geometry collision mesh filename=$(find spherorobot_cpp)/meshes/base_link.STL; visual mesh filename=$(find spherorobot_cpp)/meshes/base_link.STL
- link shaft_link: geometry collision mesh filename=$(find spherorobot_cpp)/meshes/shaft_link.STL; visual mesh filename=$(find spherorobot_cpp)/meshes/shaft_link.STL
- link sphere_link: geometry collision sphere radius=0.06; visual mesh filename=$(find spherorobot_cpp)/meshes/sphere_link.STL

File: spherorobot_cpp/urdf/spherorobot_v5_2.urdf (robot description, URDF)
Before this commit: robot spherorobot_v5_2, 3 links, 2 joints
Links:
- link base_link: geometry collision mesh filename=$(find spherorobot_cpp)/meshes/base_link.STL; visual mesh filename=$(find spherorobot_cpp)/meshes/base_link.STL
- link shaft_link: geometry collision mesh filename=$(find spherorobot_cpp)/meshes/shaft_link.STL; visual mesh filename=$(find spherorobot_cpp)/meshes/shaft_link.STL
