Commit message: work with spherorobot

File: spherorobot_cpp/urdf/spherorobot_v5_1.urdf (robot description, URDF)
Before this commit: robot spherorobot_v5_1, 3 links, 2 joints
Links:
- link base_link: mass 0.148 -> 0.177
- link sphere_link: mass 0.07 -> 0.072; geometry collision cylinder length=0.52 radius=0.06; visual mesh filename=$(find spherorobot_cpp)/meshes/sphere_link.STL
Joints:
- joint shaft_joint: child shaft_link -> base_link; parent base_link -> shaft_link
- joint sphere_joint: child sphere_link -> shaft_link; parent shaft_link -> sphere_link

File: spherorobot_cpp/urdf/vibro_table.urdf (robot description, URDF)
Before this commit: robot vibro_table, 3 links, 2 joints
Joints:
- joint left_rail_joint: origin xyz=0 0.04 0.001 rpy=0 0 0 -> xyz=0 0.05 0.001 rpy=0 0 0
- joint right_rail_joint: origin xyz=0 -0.04 0.001 rpy=0 0 0 -> xyz=0 -0.05 0.001 rpy=0 0 0

Commit message: work with sphere

File: spherorobot_cpp/urdf/spherorobot_v5_1.urdf (robot description, URDF)
Before this commit: robot spherorobot_v5_1, 3 links, 2 joints
Links:
- link base_link: mass 0.177 -> 0.148
Joints:
- joint shaft_joint: child base_link -> shaft_link; parent shaft_link -> base_link; type continuous -> fixed
- joint sphere_joint: axis 0 0 0 -> 0 1 0; child shaft_link -> sphere_link; parent sphere_link -> shaft_link; type fixed -> continuous

File: spherorobot_cpp/urdf/spherorobot_v5_2.urdf (robot description, URDF)
Before this commit: robot spherorobot_v5_2, 3 links, 2 joints
Joints:
- joint shaft_joint: type continuous -> fixed
- joint sphere_joint: axis 0 0 0 -> 0 1 0; type fixed -> continuous
