Commit message: sphero control

File: spherorobot_cpp/urdf/spherorobot_rotor_v1.urdf (robot description, URDF)
Before this commit: robot spherorobot_rotor_v1, 4 links, 3 joints
Links:
- link sphere_link: geometry collision sphere radius=0.06; visual mesh filename=$(find spherorobot_cpp)/meshes/base_sphere_link.STL
Joints:
- joint rotor_joint: axis (none) -> 0 0 -1; type fixed -> continuous
